File: PWR_Suplly/220V_AC_Supply.sch (KiCad schematic (older format))
At the start: 4 parts, among them J1 Screw_Terminal_01x02, T1 12 0- 12 1 A transformer

Commit message: uzlabotais
Parts:
- T1: value 12 0- 12 1 A transformer -> 15-0-15 transformer
Changed lines of the file:
@@
 EESchema Schematic File Version 4
+LIBS:PWR_Suplly-cache
 EELAYER 26 0
 EELAYER END
@@
 AR Path="/5C82A45A/5C828EF8" Ref="T1"  Part="1"
 F 0 "T1" H 4050 3978 50  0000 C CNN
-F 1 "12 0- 12 1 A transformer" H 4050 3887 50  0000 C CNN
+F 1 "15-0-15 transformer" H 4050 3887 50  0000 C CNN
 F 2 "" H 4050 3600 50  0001 C CNN
 F 3 "~" H 4050 3600 50  0001 C CNN

Commit message: uzlabots
Parts:
- T1: value 15-0-15 transformer -> 16-0/300mA
Changed lines of the file:
@@
 AR Path="/5C82A45A/5C828EF8" Ref="T1"  Part="1"
 F 0 "T1" H 4050 3978 50  0000 C CNN
-F 1 "15-0-15 transformer" H 4050 3887 50  0000 C CNN
+F 1 "16-0/300mA" H 4050 3887 50  0000 C CNN
 F 2 "" H 4050 3600 50  0001 C CNN
 F 3 "~" H 4050 3600 50  0001 C CNN
