File: PWR_Suplly/12V_DC_Supply.sch (KiCad schematic (older format))
At the start: 3 parts, among them U1 7805

Commit message: uzlabotais
Connections:
- wire segments 13 -> 12
Changed lines of the file:
@@
 Wire Wire Line
 	5450 3150 4850 3150
-Wire Wire Line
-	3600 2600 3500 2600
 Connection ~ 3600 2600
 Wire Wire Line
@@
 Text HLabel 5800 2600 2    50   Output ~ 0
 +12V
-Text HLabel 3150 2600 2    50   Input ~ 0
+Text HLabel 3200 2600 0    50   Input ~ 0
 VCC
-$Comp
-L power:PWR_FLAG #FLG0101
-U 1 1 5C8536CB
-P 3500 2600
-F 0 "#FLG0101" H 3500 2675 50  0001 C CNN
-F 1 "PWR_FLAG" H 3500 2774 50  0000 C CNN
-F 2 "" H 3500 2600 50  0001 C CNN
-F 3 "~" H 3500 2600 50  0001 C CNN
-	1    3500 2600
-	1    0    0    -1
-$EndComp
-Connection ~ 3500 2600
 Wire Wire Line
-	3500 2600 3200 2600
+	3200 2600 3600 2600
 $EndSCHEMATC

Commit message: uzlabots
Parts:
- removed U1: 7805, symbol Regulator_Linear:L7805
- added U1: L7812, symbol Regulator_Linear:L7812
Changed lines of the file:
@@
-	1    0    0    -1
-$EndComp
-$Comp
-L Regulator_Linear:L7805 U1
-U 1 1 5C82A8F8
-P 4850 2600
-F 0 "U1" H 4850 2842 50  0000 C CNN
-F 1 "7805" H 4850 2751 50  0000 C CNN
-F 2 "" H 4875 2450 50  0001 L CIN
-F 3 "http://www.st.com/content/ccc/resource/technical/document/datasheet/41/4f/b3/b0/12/d4/47/88/CD00000444.pdf/files/CD00000444.pdf/jcr:content/translations/en.CD00000444.pdf" H 4850 2550 50  0001 C CNN
-	1    4850 2600
 	1    0    0    -1
 $EndComp
@@
 Wire Wire Line
 	3200 2600 3600 2600
+$Comp
+L Regulator_Linear:L7812 U1
+U 1 1 5C923FFD
+P 4850 2600
+F 0 "U1" H 4850 2842 50  0000 C CNN
+F 1 "L7812" H 4850 2751 50  0000 C CNN
+F 2 "" H 4875 2450 50  0001 L CIN
+F 3 "http://www.st.com/content/ccc/resource/technical/document/datasheet/41/4f/b3/b0/12/d4/47/88/CD00000444.pdf/files/CD00000444.pdf/jcr:content/translations/en.CD00000444.pdf" H 4850 2550 50  0001 C CNN
+	1    4850 2600
+	1    0    0    -1
+$EndComp
 $EndSCHEMATC
